Commit message: add custom panda irom urdf

File: mani_skill/assets/robots/panda/panda_irom.urdf (robot description, URDF)
Before this commit: robot panda, 15 links, 14 joints
Links:
- added link camera_reference_link
- added link camera_reference_link_flipped
- link camera_link: geometry collision mesh filename=realsense2_description/meshes/wrist_mount_irom.glb; visual mesh filename=realsense2_description/meshes/wrist_mount_irom.stl
Joints:
- added joint camera_reference_joint: type fixed, parent camera_reference_link_flipped, child camera_reference_link, origin xyz=0.02 0 0 rpy=3.1415926 0 0 
- added joint camera_reference_joint_flipped: type fixed, parent panda_hand, child camera_reference_link_flipped, origin xyz=0.07422515 -0.07422515 0.0264795 rpy=0 -0.9601 2.3562
- joint panda_hand_tcp_joint: origin xyz=0 0 0.21 rpy=0 0 0 -> xyz=0 0 0.175 rpy=0 0 0
